File: Kicad/Single Int/Single Chip.kicad_sch (KiCad schematic)
At the start: 3 parts, among them J1 Raspberry_Pi_2_3, J2 Conn_01x02, U1 8088_Min_Mode

Commit message: switched back to socket
Parts:
- U1: footprint Socket:DIP_Socket-40_W11.9_W12.7_W15.24_W17.78_W18.5_3M_240-1280-00-0602J -> Package_DIP:DIP-40_W15.24mm
Changed lines of the file:
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@@
       (effects (font (size 1.27 1.27)))
     )
-    (property "Footprint" "Socket:DIP_Socket-40_W11.9_W12.7_W15.24_W17.78_W18.5_3M_240-1280-00-0602J" (at 142.24 88.9 0)
+    (property "Footprint" "Package_DIP:DIP-40_W15.24mm" (at 142.24 88.9 0)
       (effects (font (size 1.27 1.27) italic) hide)
     )
